File: driver_PCB/splitflap.kicad_pcb (KiCad board)
At the start: 2 copper layers, 19 parts, among them IC1 CD4049UBE, IC2 CD4049UBE, J1 Conn_01x02_Male, J2 Conn_01x08_Male, J3 Conn_01x16_Female, U1 74HC595, U2 74HC595, U3 SN754410NE, U4 SN754410NE, U5 SN754410NE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

Commit message: updated pcb layout
Parts:
- moved J3 254.8 mm to (254.0, 38.1)
- moved U6 185.4 mm to (209.6, 83.8), turned to 90 degrees
- moved D3 183.7 mm to (226.1, 39.4)
- moved D2 183.7 mm to (226.1, 29.2)
- moved D7 179.1 mm to (226.1, 80.0)
- moved D5 176.7 mm to (226.1, 59.7)
- moved D8 175.5 mm to (226.1, 90.2)
- moved D6 170.5 mm to (226.1, 69.8)
- moved U5 170.0 mm to (209.6, 43.2), turned to 90 degrees
- moved D4 167.3 mm to (226.1, 49.5)
- moved U4 163.3 mm to (209.6, 63.5), turned to 90 degrees
- moved D1 162.7 mm to (226.1, 19.1)
- moved U2 160.2 mm to (155.2, 70.6), turned to 90 degrees
- moved IC2 150.8 mm to (154.9, 91.4), turned to 90 degrees
- moved U3 146.9 mm to (209.6, 22.9), turned to 90 degrees
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
Commit message: updated pcb layout
Parts:
- moved IC1 1.27 mm to (156.2, 30.5)
- moved IC2 1.27 mm to (156.2, 91.4)
- moved J1 1.27 mm to (128.3, 30.5)
- moved U2 1.09 mm to (156.2, 71.1)
Changed lines of the file:
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@@
   (setup
     (last_trace_width 0.25)
+    (user_trace_width 2)
     (trace_clearance 0.2)
     (zone_clearance 0.508)
@@
   )
   (module Package_DIP:DIP-16_W7.62mm_LongPads (layer F.Cu)
-    (at 155.245001 70.604999 90)
+    (at 156.21 71.12 90)
     (descr "16-lead though-hole mounted DIP package, row spacing 7.62 mm (300 mils), LongPads")
     (tags "THT DIP DIL PDIP 2.54mm 7.62mm 300mil LongPads")
@@
   )
   (module Connector_PinSocket_2.54mm:PinSocket_1x02_P2.54mm_Vertical (layer F.Cu)
-    (at 128.27 31.75)
+    (at 128.27 30.48)
     (descr "Through hole straight socket strip, 1x02, 2.54mm pitch, single row (from Kicad 4.0.7), script generated")
     (tags "Through hole socket strip THT 1x02 2.54mm single row")
@@
   )
   (module Package_DIP:DIP-16_W7.62mm_LongPads (layer F.Cu)
-    (at 154.94 91.44 90)
+    (at 156.21 91.44 90)
     (descr "16-lead though-hole mounted DIP package, row spacing 7.62 mm (300 mils), LongPads")
     (tags "THT DIP DIL PDIP 2.54mm 7.62mm 300mil LongPads")
@@
   )
   (module Package_DIP:DIP-16_W7.62mm_LongPads (layer F.Cu)
-    (at 154.94 30.48 90)
+    (at 156.21 30.48 90)
     (descr "16-lead though-hole mounted DIP package, row spacing 7.62 mm (300 mils), LongPads")
     (tags "THT DIP DIL PDIP 2.54mm 7.62mm 300mil LongPads")

Commit message: update
Parts:
- moved J2 17.9 mm to (146.1, 48.3)
- moved J1 17.8 mm to (146.1, 30.5)
- moved J3 7.62 mm to (246.4, 38.1)
- moved IC1 3.81 mm to (160.0, 30.5)
- moved IC2 3.81 mm to (160.0, 91.4)
- moved U1 3.81 mm to (160.0, 50.8)
- moved U2 3.81 mm to (160.0, 71.1)
- moved U3 3.81 mm to (213.4, 22.9)
- moved U4 3.81 mm to (213.4, 63.5)
- moved U5 3.81 mm to (213.4, 43.2)
- moved U6 3.81 mm to (213.4, 83.8)
Connections:
- J3 pad 1: Net-(D1-Pad3) -> Net-(D1-Pad4)
- J3 pad 10: Net-(D5-Pad4) -> Net-(D5-Pad3)
- J3 pad 11: Net-(D6-Pad3) -> Net-(D6-Pad4)
- J3 pad 12: Net-(D6-Pad4) -> Net-(D6-Pad3)
- J3 pad 13: Net-(D7-Pad3) -> Net-(D7-Pad4)
- J3 pad 14: Net-(D7-Pad4) -> Net-(D7-Pad3)
- J3 pad 15: Net-(D8-Pad3) -> Net-(D8-Pad4)
- J3 pad 16: Net-(D8-Pad4) -> Net-(D8-Pad3)
- J3 pad 2: Net-(D1-Pad4) -> Net-(D1-Pad3)
- J3 pad 3: Net-(D2-Pad3) -> Net-(D2-Pad4)
- J3 pad 4: Net-(D2-Pad4) -> Net-(D2-Pad3)
- J3 pad 5: Net-(D3-Pad3) -> Net-(D3-Pad4)
- J3 pad 6: Net-(D3-Pad4) -> Net-(D3-Pad3)
- J3 pad 7: Net-(D4-Pad3) -> Net-(D4-Pad4)
- J3 pad 8: Net-(D4-Pad4) -> Net-(D4-Pad3)
- J3 pad 9: Net-(D5-Pad3) -> Net-(D5-Pad4)
- U3 pad 11: Net-(D2-Pad3) -> Net-(D2-Pad4)
- U3 pad 14: Net-(D2-Pad4) -> Net-(D2-Pad3)
- U3 pad 3: Net-(D1-Pad3) -> Net-(D1-Pad4)
- U3 pad 6: Net-(D1-Pad4) -> Net-(D1-Pad3)
- U4 pad 11: Net-(D6-Pad3) -> Net-(D6-Pad4)
- U4 pad 14: Net-(D6-Pad4) -> Net-(D6-Pad3)
- U4 pad 3: Net-(D5-Pad3) -> Net-(D5-Pad4)
- U4 pad 6: Net-(D5-Pad4) -> Net-(D5-Pad3)
- U5 pad 11: Net-(D4-Pad3) -> Net-(D4-Pad4)
- U5 pad 14: Net-(D4-Pad4) -> Net-(D4-Pad3)
- U5 pad 3: Net-(D3-Pad3) -> Net-(D3-Pad4)
- U5 pad 6: Net-(D3-Pad4) -> Net-(D3-Pad3)
- U6 pad 11: Net-(D8-Pad3) -> Net-(D8-Pad4)
- U6 pad 14: Net-(D8-Pad4) -> Net-(D8-Pad3)
- U6 pad 3: Net-(D7-Pad3) -> Net-(D7-Pad4)
- U6 pad 6: Net-(D7-Pad4) -> Net-(D7-Pad3)
Routing:
- net Net-(D1-Pad4): track 0.00 -> 30.3 mm
- net Net-(D8-Pad3): track 0.00 -> 30.3 mm
- net Net-(D1-Pad3): track 0.00 -> 27.7 mm
- net Net-(D8-Pad4): track 0.00 -> 26.2 mm
- net Net-(D2-Pad4): track 0.00 -> 23.0 mm
- net Net-(D7-Pad3): track 0.00 -> 23.0 mm
- net Net-(D2-Pad3): track 0.00 -> 20.4 mm
- net Net-(D7-Pad4): track 0.00 -> 19.7 mm
- net Net-(D6-Pad3): track 0.00 -> 16.4 mm
- net Net-(D3-Pad4): track 0.00 -> 16.4 mm
- net Net-(D6-Pad4): track 0.00 -> 15.3 mm
- net Net-(D3-Pad3): track 0.00 -> 15.3 mm
- net Net-(D4-Pad4): track 0.00 -> 14.3 mm
- net Net-(D5-Pad3): track 0.00 -> 14.3 mm
- net Net-(D4-Pad3): track 0.00 -> 13.2 mm
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