File: driver_PCB/splitflap.sch (KiCad schematic (older format))
At the start: 25 parts

Commit message: updated kicad schematic
Parts:
- removed U? (x8): 4049, symbol 4xxx:4049
- added IC1, IC2: CD4049UBE, Package_DIP:DIP-16_W7.62mm_LongPads, symbol CD4049UBE:CD4049UBE
- D1, D2, D3, D4, D5, D6, D7, D8: renamed from D?; footprint (none) -> Diode_THT:Diode_Bridge_DIP-4_W7.62mm_P5.08mm
- J1: renamed from J?; footprint (none) -> Connector_PinSocket_2.54mm:PinSocket_1x02_P2.54mm_Vertical
- J2: renamed from J?; footprint (none) -> Connector_PinSocket_2.54mm:PinSocket_1x08_P2.54mm_Vertical
- J3: renamed from J?; footprint (none) -> Connector_PinSocket_2.54mm:PinSocket_1x16_P2.54mm_Vertical
- U1, U2: renamed from U?; footprint (none) -> Package_DIP:DIP-16_W7.62mm_LongPads
- gave numbers to parts that had none: 4
Connections:
- wire segments 371 -> 400

Commit message: update
Connections:
- net at J3.3 (Pin_3), U3.11 (3Y): now also D2.4 (~~); no longer D2.3 (~~)
- net at J3.4 (Pin_4), U3.14 (4Y): now also D2.3 (~~); no longer D2.4 (~~)
- net at J3.1 (Pin_1), U3.3 (1Y): now also D1.4 (~~); no longer D1.3 (~~)
- net at J3.2 (Pin_2), U3.6 (2Y): now also D1.3 (~~); no longer D1.4 (~~)
- net at J3.11 (Pin_11), U4.11 (3Y): now also D6.4 (~~); no longer D6.3 (~~)
- net at J3.12 (Pin_12), U4.14 (4Y): now also D6.3 (~~); no longer D6.4 (~~)
- net at J3.9 (Pin_9), U4.3 (1Y): now also D5.4 (~~); no longer D5.3 (~~)
- net at J3.10 (Pin_10), U4.6 (2Y): now also D5.3 (~~); no longer D5.4 (~~)
- net at J3.7 (Pin_7), U5.11 (3Y): now also D4.4 (~~); no longer D4.3 (~~)
- net at J3.8 (Pin_8), U5.14 (4Y): now also D4.3 (~~); no longer D4.4 (~~)
- net at J3.5 (Pin_5), U5.3 (1Y): now also D3.4 (~~); no longer D3.3 (~~)
- net at J3.6 (Pin_6), U5.6 (2Y): now also D3.3 (~~); no longer D3.4 (~~)
- net at J3.15 (Pin_15), U6.11 (3Y): now also D8.4 (~~); no longer D8.3 (~~)
- net at J3.16 (Pin_16), U6.14 (4Y): now also D8.3 (~~); no longer D8.4 (~~)
- net at J3.13 (Pin_13), U6.3 (1Y): now also D7.4 (~~); no longer D7.3 (~~)
- net at J3.14 (Pin_14), U6.6 (2Y): now also D7.3 (~~); no longer D7.4 (~~)
Changed lines of the file:
@@
 F 3 "~" H 12750 2200 50  0001 C CNN
 	1    12750 2200
-	1    0    0    -1
+	1    0    0    1
 $EndComp
 $Comp
@@
 F 3 "~" H 12750 2900 50  0001 C CNN
 	1    12750 2900
-	1    0    0    -1
+	1    0    0    1
 $EndComp
 $Comp
@@
 F 3 "~" H 12750 3600 50  0001 C CNN
 	1    12750 3600
-	1    0    0    -1
+	1    0    0    1
 $EndComp
 $Comp
@@
 F 3 "~" H 12750 5700 50  0001 C CNN
 	1    12750 5700
-	1    0    0    -1
+	1    0    0    1
 $EndComp
 $Comp
@@
 F 3 "~" H 12750 6400 50  0001 C CNN
 	1    12750 6400
-	1    0    0    -1
+	1    0    0    1
 $EndComp
 $Comp
@@
 F 3 "~" H 12750 7100 50  0001 C CNN
 	1    12750 7100
-	1    0    0    -1
+	1    0    0    1
 $EndComp
 $Comp
@@
 F 3 "~" H 12750 5000 50  0001 C CNN
 	1    12750 5000
-	1    0    0    -1
+	1    0    0    1
 $EndComp
 $Comp
@@
 F 3 "~" H 12750 4300 50  0001 C CNN
 	1    12750 4300
-	1    0    0    -1
+	1    0    0    1
 $EndComp
 Wire Wire Line
