File: hardware/driver_PCB/_autosave-splitflap.kicad_pcb (KiCad board)
At the start: 2 copper layers, 111.8 x 95.2 mm, 19 parts, among them IC1 CD4049UBE, IC2 CD4049UBE, J1 Conn_01x02_Male, J2 Conn_01x08_Male, J3 Conn_01x16_Female, U1 74HC595, U2 74HC595, U3 SN754410NE, U4 SN754410NE, U5 SN754410NE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

Commit message: update
Routing:
- net GND: vias 23 -> 25
Changed lines of the file:
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@@
     (thickness 1.6)
     (drawings 7)
-    (tracks 635)
+    (tracks 637)
     (zones 0)
     (modules 19)
@@
   (via (at 222.25 87.63) (size 0.8) (drill 0.4) (layers F.Cu B.Cu) (net 3))
   (via (at 222.25 67.31) (size 0.8) (drill 0.4) (layers F.Cu B.Cu) (net 3))
+  (via (at 163.83 74.93) (size 0.8) (drill 0.4) (layers F.Cu B.Cu) (net 3))
+  (via (at 217.17 73.66) (size 0.8) (drill 0.4) (layers F.Cu B.Cu) (net 3))
   (segment (start 233.68 35.56) (end 243.84 35.56) (width 0.25) (layer F.Cu) (net 4))
   (segment (start 246.38 38.1) (end 246.38 54.61) (width 0.25) (layer F.Cu) (net 4))
