File: hardware/driver_PCB/splitflap.sch (KiCad schematic (older format))
At the start: 19 parts, among them IC1 CD4049UBE, IC2 CD4049UBE, J1 Conn_01x02_Male, J2 Conn_01x08_Male, J3 Conn_01x16_Female, U1 74HC595, U2 74HC595, U3 SN754410NE, U4 SN754410NE, U5 SN754410NE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

Commit message: finished pcb layout
Parts:
- IC1, IC2: symbol CD4049UBE:CD4049UBE -> splitflap-rescue:CD4049UBE-CD4049UBE
Changed lines of the file:
@@
 F 3 "~" H 12750 2200 50  0001 C CNN
 	1    12750 2200
-	1    0    0    -1
+	1    0    0    1
 $EndComp
 $Comp
@@
 F 3 "~" H 12750 2900 50  0001 C CNN
 	1    12750 2900
-	1    0    0    -1
+	1    0    0    1
 $EndComp
 $Comp
@@
 F 3 "~" H 12750 3600 50  0001 C CNN
 	1    12750 3600
-	1    0    0    -1
+	1    0    0    1
 $EndComp
 $Comp
@@
 F 3 "~" H 12750 5700 50  0001 C CNN
 	1    12750 5700
-	1    0    0    -1
+	1    0    0    1
 $EndComp
 $Comp
@@
 F 3 "~" H 12750 6400 50  0001 C CNN
 	1    12750 6400
-	1    0    0    -1
+	1    0    0    1
 $EndComp
 $Comp
@@
 F 3 "~" H 12750 7100 50  0001 C CNN
 	1    12750 7100
-	1    0    0    -1
+	1    0    0    1
 $EndComp
 $Comp
@@
 F 3 "~" H 12750 5000 50  0001 C CNN
 	1    12750 5000
-	1    0    0    -1
+	1    0    0    1
 $EndComp
 $Comp
@@
 F 3 "~" H 12750 4300 50  0001 C CNN
 	1    12750 4300
-	1    0    0    -1
+	1    0    0    1
 $EndComp
 Wire Wire Line
@@
 	2300 4800 1000 4800
 $Comp
-L CD4049UBE:CD4049UBE IC2
+L splitflap-rescue:CD4049UBE-CD4049UBE IC2
 U 1 1 5E1254E2
 P 5350 3400
@@
 	5100 1600 5100 2450
 $Comp
-L CD4049UBE:CD4049UBE IC1
+L splitflap-rescue:CD4049UBE-CD4049UBE IC1
 U 1 1 5DED8412
 P 5200 1950

Commit message: changed pcb layout and interface
Parts:
- removed J1: Conn_01x02_Male, Connector_PinSocket_2.54mm:PinSocket_1x02_P2.54mm_Vertical, symbol Connector:Conn_01x02_Male
- removed J2: Conn_01x08_Male, Connector_PinSocket_2.54mm:PinSocket_1x08_P2.54mm_Vertical, symbol Connector:Conn_01x08_Male
- added J1, J2: Conn_02x06_Odd_Even, Connector_PinSocket_2.54mm:PinSocket_2x06_P2.54mm_Vertical, symbol Connector_Generic:Conn_02x06_Odd_Even
- U3, U4, U5, U6: footprint DIP254P762X508-16 -> Package_DIP:DIP-16_W7.62mm_LongPads; symbol SN754410NE:SN754410NE -> splitflap-rescue:SN754410NE-SN754410NE
Connections:
- net GND: now also J1.11 (Pin_11), J1.12 (Pin_12), J2.11 (Pin_11), J2.12 (Pin_12)
- net VCC: now also J1.3 (Pin_3), J1.4 (Pin_4), J2.3 (Pin_3), J2.4 (Pin_4)
- net VDD: now also J1.1 (Pin_1), J1.2 (Pin_2), J2.1 (Pin_1), J2.2 (Pin_2)
- net at U2.11 (SRCLK): now also J1.8 (Pin_8), J2.8 (Pin_8)
- net at U2.12 (RCLK): now also J1.10 (Pin_10), J2.10 (Pin_10)
- net at U2.14 (SER): now also J1.6 (Pin_6)
- net at U2.9 (QH'): now also J2.6 (Pin_6)
- net at U1.11 (SRCLK): now also J1.7 (Pin_7), J2.7 (Pin_7)
- net at U1.12 (RCLK): now also J1.9 (Pin_9), J2.9 (Pin_9)
- net at U1.14 (SER): now also J1.5 (Pin_5)
- net at U1.9 (QH'): now also J2.5 (Pin_5)
