File: hardware/driver_PCB/splitflap.sch (KiCad schematic (older format))
At the start: 34 parts, among them IC1 CD4049UBE, IC2 CD4049UBE, J1 Conn_02x06_Odd_Even, J2 Conn_02x06_Odd_Even, J3 Screw_Terminal_01x04, J4 Screw_Terminal_01x04, J5 Screw_Terminal_01x04, J6 Screw_Terminal_01x04, U1 74HC595, U2 74HC595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

Commit message: idk
Parts:
- added J7: Screw_Terminal_01x02, TerminalBlock:TerminalBlock_bornier-2_P5.08mm, symbol Connector:Screw_Terminal_01x02
- C1, C10, C11, C12, C2, C3, C4, C5, C6, C7, C8, C9: symbol Device:CP -> splitflap-rescue:CP-Device
- D1, D2, D3, D4, D5, D6, D7, D8: symbol Device:D_Bridge_+-AA -> splitflap-rescue:D_Bridge_+-AA-Device
- IC1, IC2: symbol splitflap-rescue:CD4049UBE-CD4049UBE -> splitflap-rescue:CD4049UBE-CD4049UBE-splitflap-rescue
- J1, J2: symbol Connector_Generic:Conn_02x06_Odd_Even -> splitflap-rescue:Conn_02x06_Odd_Even-Connector_Generic
- J3, J4, J5, J6: symbol Connector:Screw_Terminal_01x04 -> splitflap-rescue:Screw_Terminal_01x04-Connector
- U1, U2: symbol 74xx:74HC595 -> splitflap-rescue:74HC595-74xx
- U3, U4, U5, U6: symbol splitflap-rescue:SN754410NE-SN754410NE -> splitflap-rescue:SN754410NE-SN754410NE-splitflap-rescue
Connections:
- net labels added: GND-power
- wire segments 527 -> 532
Other:
- moved on the sheet: D1, D2, D3, D4, D5, D6, D7, D8, IC1, IC2, J1, J2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
