File: hardware/driver_PCB/splitflap.kicad_pcb (KiCad board)
At the start: 2 copper layers, 111.8 x 95.2 mm, 19 parts, among them IC1 CD4049UBE, IC2 CD4049UBE, J1 Conn_02x06_Odd_Even, J2 Conn_02x06_Odd_Even, J3 Conn_01x16_Female, U1 74HC595, U2 74HC595, U3 SN754410NE, U4 SN754410NE, U5 SN754410NE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

Commit message: updated pcb
Parts:
- added C1: CP, Capacitor_THT:CP_Radial_D4.0mm_P2.00mm, F.Cu at (208.9, 53.3)
- added C10: CP, Capacitor_THT:CP_Radial_D4.0mm_P2.00mm, F.Cu at (208.9, 94.0)
- added C11: CP, Capacitor_THT:CP_Radial_D6.3mm_P2.50mm, F.Cu at (200.0, 33.7)
- added C12: CP, Capacitor_THT:CP_Radial_D6.3mm_P2.50mm, F.Cu at (200.0, 94.6)
- added C2: CP, Capacitor_THT:CP_Radial_D4.0mm_P2.00mm, F.Cu at (176.4, 95.9)
- added C3: CP, Capacitor_THT:CP_Radial_D4.0mm_P2.00mm, F.Cu at (176.4, 55.2)
- added C4: CP, Capacitor_THT:CP_Radial_D4.0mm_P2.00mm, F.Cu at (208.9, 73.7)
- added C5: CP, Capacitor_THT:CP_Radial_D6.3mm_P2.50mm, F.Cu at (200.0, 54.0)
- added C6: CP, Capacitor_THT:CP_Radial_D4.0mm_P2.00mm, F.Cu at (208.9, 34.3)
- added C7: CP, Capacitor_THT:CP_Radial_D4.0mm_P2.00mm, F.Cu at (176.4, 75.6)
- added C8: CP, Capacitor_THT:CP_Radial_D6.3mm_P2.50mm, F.Cu at (200.0, 74.3)
- added C9: CP, Capacitor_THT:CP_Radial_D4.0mm_P2.00mm, F.Cu at (176.5, 34.9)
- added G***: LOGO, maldegem:logo_maldegem2, F.Cu at (214.6, 114.3)
- added J4: Screw_Terminal_01x04, TerminalBlock:TerminalBlock_bornier-4_P5.08mm, F.Cu at (236.2, 55.2)
- added J5: Screw_Terminal_01x04, TerminalBlock:TerminalBlock_bornier-4_P5.08mm, F.Cu at (236.2, 76.8)
- added J6: Screw_Terminal_01x04, TerminalBlock:TerminalBlock_bornier-4_P5.08mm, F.Cu at (236.2, 98.4)
- added REF**: MountingHole_3.2mm_M3, MountingHole2:MountingHole_3.2mm_M3, F.Cu at (250.0, 113.0)
- added REF**: MountingHole_3.2mm_M3, MountingHole2:MountingHole_3.2mm_M3, F.Cu at (160.0, 113.0)
- added REF**: MountingHole_3.2mm_M3, MountingHole2:MountingHole_3.2mm_M3, F.Cu at (250.0, 33.0)
- added REF**: MountingHole_3.2mm_M3, MountingHole2:MountingHole_3.2mm_M3, F.Cu at (160.0, 33.0)
- INPUT: renamed from J1; footprint Connector_PinSocket_2.54mm:PinSocket_2x06_P2.54mm_Vertical -> Connector_IDC:IDC-Header_2x06_P2.54mm_Vertical
- J2: footprint Connector_PinSocket_2.54mm:PinSocket_2x06_P2.54mm_Vertical -> Connector_IDC:IDC-Header_2x06_P2.54mm_Vertical
- J3: value Conn_01x16_Female -> Screw_Terminal_01x04; footprint Connector_PinSocket_2.54mm:PinSocket_1x16_P2.54mm_Vertical -> TerminalBlock:TerminalBlock_bornier-4_P5.08mm
- moved J3 23.3 mm to (236.2, 33.7), turned to 270 degrees
- moved D1 5.08 mm to (221.0, 35.6)
- moved D2 5.08 mm to (221.0, 45.7)
- moved D3 5.08 mm to (221.0, 55.9)
- moved D4 5.08 mm to (221.0, 66.0)
- moved D5 5.08 mm to (221.0, 76.2)
- moved D6 5.08 mm to (221.0, 86.4)
- moved D7 5.08 mm to (221.0, 96.5)
- moved D8 5.08 mm to (221.0, 106.7)
- moved IC1 5.08 mm to (170.2, 47.0)
- moved IC2 5.08 mm to (170.2, 108.0)
- moved INPUT 5.08 mm to (156.2, 54.6)
- moved J2 5.08 mm to (156.2, 80.0)
- moved U1 5.08 mm to (170.2, 67.3)
- moved U2 5.08 mm to (170.2, 87.6)
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Routing:
- net VCC: track 356.1 -> 443.1 mm
- net Net-(J2-Pad6): track 53.7 -> 32.3 mm, vias 1 -> 0
- net Net-(D8-Pad3): track 48.5 -> 32.6 mm
- net Net-(D1-Pad4): track 48.5 -> 32.6 mm
- net Net-(D8-Pad4): track 53.6 -> 38.7 mm
- net Net-(D1-Pad3): track 53.6 -> 38.7 mm
- net Net-(J1-Pad7): track 56.1 -> 69.7 mm, vias 0 -> 1
- net Net-(D7-Pad3): track 51.8 -> 38.7 mm
- net Net-(D2-Pad4): track 51.8 -> 38.7 mm
- net Net-(D2-Pad3): track 43.9 -> 32.6 mm
- net Net-(D7-Pad4): track 43.7 -> 32.4 mm
- net Net-(IC1-Pad11): track 137.0 -> 148.0 mm
- net Net-(D3-Pad4): track 42.3 -> 32.1 mm
- net Net-(D6-Pad3): track 41.9 -> 31.9 mm
- net Net-(J1-Pad9): track 55.2 -> 64.6 mm, vias 0 -> 1
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Other:
- board text added: "Clk"
- board text added: "ClkE"
- board text added: "D"
- board text added: "DE"
- board text added: "La"
- board text added: "LaE"
- board text added: "brainchild of Dylan Missuwe"
- board text removed: "A1"
- board text removed: "A2"
- board text removed: "A3"
- board text removed: "A4"
- board text removed: "A5"
- board text removed: "A6"
- board text removed: "A7"
- board text removed: "A8"
- board text removed: "B1"
- board text removed: "B2"
- board text removed: "B3"
- board text removed: "B4"
- board text removed: "B5"
- board text removed: "B6"
- board text removed: "B7"
- board text removed: "B8"
- board text removed: "Clock"
- board text removed: "Clock-EN"
- board text removed: "Data"
- board text removed: "Data-EN"
- board text removed: "INPUT"
- board text removed: "Latch"
- board text removed: "Latch-EN"

Commit message: update
Routing:
- net VCC: track 443.1 -> 443.7 mm
- net GND: vias 64 -> 113
Changed lines of the file:
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@@
     (thickness 1.6)
     (drawings 47)
-    (tracks 830)
+    (tracks 878)
     (zones 0)
     (modules 39)
@@
   )
   (setup
-    (last_trace_width 2)
+    (last_trace_width 0.25)
     (user_trace_width 0.5)
     (user_trace_width 1)
@@
   (via (at 186.69 41.91) (size 0.8) (drill 0.4) (layers F.Cu B.Cu) (net 3))
   (via (at 187.96 41.91) (size 0.8) (drill 0.4) (layers F.Cu B.Cu) (net 3))
-  (via (at 204.47 35.56) (size 0.8) (drill 0.4) (layers F.Cu B.Cu) (net 3))
   (via (at 203.2 35.56) (size 0.8) (drill 0.4) (layers F.Cu B.Cu) (net 3))
-  (via (at 207.01 35.56) (size 0.8) (drill 0.4) (layers F.Cu B.Cu) (net 3))
+  (via (at 204.47 36.83) (size 0.8) (drill 0.4) (layers F.Cu B.Cu) (net 3))
+  (via (at 205.74 35.56) (size 0.8) (drill 0.4) (layers F.Cu B.Cu) (net 3))
   (via (at 204.47 45.72) (size 0.8) (drill 0.4) (layers F.Cu B.Cu) (net 3))
   (via (at 179.07 41.91) (size 0.8) (drill 0.4) (layers F.Cu B.Cu) (net 3))
@@
   (via (at 226.06 34.29) (size 0.8) (drill 0.4) (layers F.Cu B.Cu) (net 3))
   (via (at 226.06 33.02) (size 0.8) (drill 0.4) (layers F.Cu B.Cu) (net 3))
+  (via (at 204.47 60.96) (size 0.8) (drill 0.4) (layers F.Cu B.Cu) (net 3))
+  (via (at 204.47 58.42) (size 0.8) (drill 0.4) (layers F.Cu B.Cu) (net 3))
+  (via (at 204.47 58.42) (size 0.8) (drill 0.4) (layers F.Cu B.Cu) (net 3))
+  (via (at 207.01 69.85) (size 0.8) (drill 0.4) (layers F.Cu B.Cu) (net 3))
+  (via (at 205.74 69.85) (size 0.8) (drill 0.4) (layers F.Cu B.Cu) (net 3))
+  (via (at 204.47 69.85) (size 0.8) (drill 0.4) (layers F.Cu B.Cu) (net 3))
+  (via (at 203.2 69.85) (size 0.8) (drill 0.4) (layers F.Cu B.Cu) (net 3))
+  (via (at 201.93 69.85) (size 0.8) (drill 0.4) (layers F.Cu B.Cu) (net 3))
+  (via (at 203.2 36.83) (size 0.8) (drill 0.4) (layers F.Cu B.Cu) (net 3))
+  (via (at 205.74 36.83) (size 0.8) (drill 0.4) (layers F.Cu B.Cu) (net 3))
+  (via (at 204.47 35.56) (size 0.8) (drill 0.4) (layers F.Cu B.Cu) (net 3))
+  (via (at 207.01 36.83) (size 0.8) (drill 0.4) (layers F.Cu B.Cu) (net 3))
+  (via (at 201.93 36.83) (size 0.8) (drill 0.4) (layers F.Cu B.Cu) (net 3))
+  (via (at 205.74 40.64) (size 0.8) (drill 0.4) (layers F.Cu B.Cu) (net 3))
+  (via (at 204.47 40.64) (size 0.8) (drill 0.4) (layers F.Cu B.Cu) (net 3))
+  (via (at 201.93 49.53) (size 0.8) (drill 0.4) (layers F.Cu B.Cu) (net 3))
+  (via (at 203.2 49.53) (size 0.8) (drill 0.4) (layers F.Cu B.Cu) (net 3))
+  (via (at 204.47 49.53) (size 0.8) (drill 0.4) (layers F.Cu B.Cu) (net 3))
+  (via (at 205.74 49.53) (size 0.8) (drill 0.4) (layers F.Cu B.Cu) (net 3))
+  (via (at 207.01 49.53) (size 0.8) (drill 0.4) (layers F.Cu B.Cu) (net 3))
+  (via (at 205.74 50.8) (size 0.8) (drill 0.4) (layers F.Cu B.Cu) (net 3))
+  (via (at 204.47 50.8) (size 0.8) (drill 0.4) (layers F.Cu B.Cu) (net 3))
+  (via (at 203.2 50.8) (size 0.8) (drill 0.4) (layers F.Cu B.Cu) (net 3))
+  (via (at 203.2 71.12) (size 0.8) (drill 0.4) (layers F.Cu B.Cu) (net 3))
+  (via (at 204.47 71.12) (size 0.8) (drill 0.4) (layers F.Cu B.Cu) (net 3))
+  (via (at 205.74 71.12) (size 0.8) (drill 0.4) (layers F.Cu B.Cu) (net 3))
+  (via (at 205.74 77.47) (size 0.8) (drill 0.4) (layers F.Cu B.Cu) (net 3))
+  (via (at 204.47 77.47) (size 0.8) (drill 0.4) (layers F.Cu B.Cu) (net 3))
+  (via (at 203.2 77.47) (size 0.8) (drill 0.4) (layers F.Cu B.Cu) (net 3))
+  (via (at 207.01 77.47) (size 0.8) (drill 0.4) (layers F.Cu B.Cu) (net 3))
+  (via (at 201.93 77.47) (size 0.8) (drill 0.4) (layers F.Cu B.Cu) (net 3))
+  (via (at 204.47 81.28) (size 0.8) (drill 0.4) (layers F.Cu B.Cu) (net 3))
+  (via (at 205.74 81.28) (size 0.8) (drill 0.4) (layers F.Cu B.Cu) (net 3))
+  (via (at 205.74 91.44) (size 0.8) (drill 0.4) (layers F.Cu B.Cu) (net 3))
+  (via (at 204.47 91.44) (size 0.8) (drill 0.4) (layers F.Cu B.Cu) (net 3))
+  (via (at 203.2 91.44) (size 0.8) (drill 0.4) (layers F.Cu B.Cu) (net 3))
+  (via (at 205.74 97.79) (size 0.8) (drill 0.4) (layers F.Cu B.Cu) (net 3))
+  (via (at 204.47 97.79) (size 0.8) (drill 0.4) (layers F.Cu B.Cu) (net 3))
+  (via (at 203.2 97.79) (size 0.8) (drill 0.4) (layers F.Cu B.Cu) (net 3))
+  (via (at 201.93 97.79) (size 0.8) (drill 0.4) (layers F.Cu B.Cu) (net 3))
+  (via (at 207.01 97.79) (size 0.8) (drill 0.4) (layers F.Cu B.Cu) (net 3))
+  (via (at 207.01 110.49) (size 0.8) (drill 0.4) (layers F.Cu B.Cu) (net 3))
+  (via (at 205.74 110.49) (size 0.8) (drill 0.4) (layers F.Cu B.Cu) (net 3))
+  (via (at 204.47 110.49) (size 0.8) (drill 0.4) (layers F.Cu B.Cu) (net 3))
+  (via (at 203.2 110.49) (size 0.8) (drill 0.4) (layers F.Cu B.Cu) (net 3))
+  (via (at 201.93 110.49) (size 0.8) (drill 0.4) (layers F.Cu B.Cu) (net 3))
+  (via (at 203.2 111.76) (size 0.8) (drill 0.4) (layers F.Cu B.Cu) (net 3))
+  (via (at 204.47 111.76) (size 0.8) (drill 0.4) (layers F.Cu B.Cu) (net 3))
+  (via (at 205.74 111.76) (size 0.8) (drill 0.4) (layers F.Cu B.Cu) (net 3))
   (segment (start 228.6 35.56) (end 222.25 41.91) (width 0.5) (layer B.Cu) (net 4))
   (segment (start 222.25 41.91) (end 210.42 41.91) (width 0.5) (layer B.Cu) (net 4))
@@
   (segment (start 172.41499 61.26501) (end 168.504989 65.175011) (width 0.25) (layer F.Cu) (net 33))
   (segment (start 172.97501 61.26501) (end 172.41499 61.26501) (width 0.25) (layer F.Cu) (net 33))
-  (segment (start 193.726062 43.214942) (end 196.94499 39.996014) (width 0.25) (layer F.Cu) (net 33))
-  (segment (start 173.555058 43.214942) (end 193.726062 43.214942) (width 0.25) (layer F.Cu) (net 33))
+  (segment (start 208.89001 37.79499) (end 209.855 36.83) (width 0.25) (layer F.Cu) (net 33))
+  (segment (start 196.94499 38.483295) (end 197.633295 37.79499) (width 0.25) (layer F.Cu) (net 33))
   (segment (start 170.18 46.99) (end 170.18 46.59) (width 0.25) (layer F.Cu) (net 33))
-  (segment (start 197.633295 37.79499) (end 203.50501 37.79499) (width 0.25) (layer F.Cu) (net 33))
-  (segment (start 196.94499 39.996014) (end 196.94499 38.483295) (width 0.25) (layer F.Cu) (net 33))
+  (segment (start 197.633295 37.79499) (end 208.89001 37.79499) (width 0.25) (layer F.Cu) (net 33))
+  (segment (start 173.555058 43.214942) (end 193.726062 43.214942) (width 0.25) (layer F.Cu) (net 33))
   (segment (start 170.18 46.59) (end 173.555058 43.214942) (width 0.25) (layer F.Cu) (net 33))
-  (segment (start 196.94499 38.483295) (end 197.633295 37.79499) (width 0.25) (layer F.Cu) (net 33))
-  (segment (start 203.50501 37.79499) (end 204.47 36.83) (width 0.25) (layer F.Cu) (net 33))
-  (segment (start 207.975 36.83) (end 208.915 35.89) (width 0.25) (layer F.Cu) (net 33))
-  (segment (start 204.47 36.83) (end 207.975 36.83) (width 0.25) (layer F.Cu) (net 33))
+  (segment (start 193.726062 43.214942) (end 196.94499 39.996014) (width 0.25) (layer F.Cu) (net 33))
+  (segment (start 196.94499 39.996014) (end 196.94499 38.483295) (width 0.25) (layer F.Cu) (net 33))
   (segment (start 198.12 107.55) (end 198.12 107.95) (width 0.25) (layer F.Cu) (net 38))
   (segment (start 196.99499 106.42499) (end 198.12 107.55) (width 0.25) (layer F.Cu) (net 38))
@@
   (segment (start 189.23 71.12) (end 190.5 72.39) (width 0.25) (layer B.Cu) (net 48))
   (segment (start 186.29 71.12) (end 189.23 71.12) (width 0.25) (layer B.Cu) (net 48))
-  (segment (start 213.36 99.93) (end 211.855 98.425) (width 0.25) (layer B.Cu) (net 48))
   (segment (start 213.36 100.33) (end 213.36 99.93) (width 0.25) (layer B.Cu) (net 48))
-  (segment (start 211.855 98.425) (end 196.215 98.425) (width 0.25) (layer B.Cu) (net 48))
-  (segment (start 194.945 97.155) (end 194.945 89.353305) (width 0.25) (layer B.Cu) (net 48))
-  (segment (start 196.215 98.425) (end 194.945 97.155) (width 0.25) (layer B.Cu) (net 48))
-  (segment (start 194.945 89.353305) (end 190.5 84.908305) (width 0.25) (layer B.Cu) (net 48))
   (segment (start 190.5 72.39) (end 190.5 83.82) (width 0.25) (layer B.Cu) (net 48))
-  (segment (start 190.5 84.908305) (end 190.5 83.82) (width 0.25) (layer B.Cu) (net 48))
   (segment (start 190.5 83.82) (end 190.5 84.611715) (width 0.25) (layer B.Cu) (net 48))
+  (segment (start 194.945 89.353305) (end 190.5 84.908305) (width 0.25) (layer B.Cu) (net 48))
+  (segment (start 213.36 97.79) (end 212.09 96.52) (width 0.25) (layer B.Cu) (net 48))
+  (segment (start 190.5 84.908305) (end 190.5 83.82) (width 0.25) (layer B.Cu) (net 48))
+  (segment (start 213.36 100.33) (end 213.36 97.79) (width 0.25) (layer B.Cu) (net 48))
+  (segment (start 212.09 96.52) (end 196.85 96.52) (width 0.25) (layer B.Cu) (net 48))
+  (segment (start 196.85 96.52) (end 194.945 94.615) (width 0.25) (layer B.Cu) (net 48))
+  (segment (start 194.945 94.615) (end 194.945 89.353305) (width 0.25) (layer B.Cu) (net 48))
   (segment (start 180.34 67.31) (end 180.34 67.71) (width 0.25) (layer F.Cu) (net 49))
   (via (at 190.5 69.85) (size 0.8) (drill 0.4) (layers F.Cu B.Cu) (net 49))
@@
   (segment (start 175.26 59.69) (end 175.26 60.09) (width 0.25) (layer B.Cu) (net 59))
   (zone (net 3) (net_name GND) (layer B.Cu) (hatch edge 0.508)
-    (connect_pads (clearance 0.508))
+    (connect_pads yes (clearance 0.508))
     (min_thickness 0.254)
     (fill yes (arc_segments 32) (thermal_gap 0.508) (thermal_bridge_width 0.508))
@@
   )
   (zone (net 3) (net_name GND) (layer F.Cu) (hatch edge 0.508)
-    (connect_pads (clearance 0.508))
+    (connect_pads yes (clearance 0.508))
     (min_thickness 0.254)
     (fill yes (arc_segments 32) (thermal_gap 0.508) (thermal_bridge_width 0.508))
