File: hardware/driver_PCB/splitflap.kicad_pcb (KiCad board)
At the start: 2 copper layers, 111.8 x 95.2 mm, 39 parts, among them IC1 CD4049UBE, IC2 CD4049UBE, J2 Conn_02x06_Odd_Even, J3 Screw_Terminal_01x04, J4 Screw_Terminal_01x04, J5 Screw_Terminal_01x04, J6 Screw_Terminal_01x04, U1 74HC595, U2 74HC595, U3 SN754410NE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

Commit message: converted arduino sketch to a library ann pcb updates
Parts:
- moved REF** 5.08 mm to (244.9, 113.0)
- moved REF** 5.08 mm to (154.9, 113.0)
- moved REF** 5.08 mm to (244.9, 33.0)
- moved REF** 5.08 mm to (154.9, 33.0)
Other:
- board text added: "A0"
- board text added: "A1"
- board text added: "A2"
- board text added: "A3"
- board text added: "A4"
- board text added: "A5"
- board text added: "A6"
- board text added: "A7"
- board text added: "B0"
- board text added: "B1"
- board text added: "B2"
- board text added: "B3"
- board text added: "B4"
- board text added: "B5"
- board text added: "B6"
- board text added: "B7"

Commit message: idk
Parts:
- removed the REF** at (244.9, 113.0)
- removed the REF** at (154.9, 113.0)
- added J7: Screw_Terminal_01x02, TerminalBlock:TerminalBlock_bornier-2_P5.08mm, F.Cu at (160.7, 98.4)
- INPUT J1: renamed from INPUT
- OUTPUT J2: renamed from J2
- moved C6 80.0 mm to (208.9, 114.3)
- moved G*** 12.1 mm to (202.6, 114.3)
- moved OUTPUT J2 11.4 mm to (156.2, 68.6)
- moved INPUT J1 11.4 mm to (156.2, 43.2)
Routing:
- net VDD: track 295.5 -> 318.3 mm
- net Net-(J1-Pad5): track 22.0 -> 42.5 mm
- net Net-(J1-Pad7): track 69.7 -> 84.9 mm
- net Net-(J2-Pad5): track 55.2 -> 64.0 mm
- net Net-(J1-Pad6): track 32.6 -> 40.3 mm
- net Net-(J1-Pad8): track 66.7 -> 61.4 mm
- net Net-(J1-Pad9): track 64.6 -> 60.5 mm
- net Net-(J1-Pad10): track 65.5 -> 67.8 mm
- net VCC: track 443.7 -> 442.4 mm
- net GND: vias 118 -> 128
Other:
- board text added: "+Vdd"
- board text added: "Di"
- board text added: "DiE"
- board text added: "Do"
- board text added: "DoE"
- board text added: "brainchild of Dylan Missuwe and Tijl Desmet"
- board text removed: "D"
- board text removed: "DE"
- board text removed: "OUTPUT"
- board text removed: "brainchild of Dylan Missuwe"
