File: hardware/main_pcb/splitflap.sch (KiCad schematic (older format))
At the start: 10 parts, among them J1 Conn_02x06_Odd_Even, J2 Conn_02x06_Odd_Even, J3 Conn_02x06_Odd_Even, J4 Conn_02x06_Odd_Even, J5 Conn_02x06_Odd_Even, J6 Conn_02x06_Odd_Even, J7 Conn_02x06_Odd_Even, J8 Conn_02x06_Odd_Even

Commit message: updated splitflap library
Parts:
- removed J3, J6: Conn_02x06_Odd_Even, Connector_IDC:IDC-Header_2x06_P2.54mm_Vertical, symbol Connector_Generic:Conn_02x06_Odd_Even
- added 1.6k, 1k, 280R: R, symbol Device:R
- added D? (x3): LED, symbol Device:LED
- added J?: Screw_Terminal_01x04, symbol Connector:Screw_Terminal_01x04
- added J?: Conn_01x02_Female, symbol Connector:Conn_01x02_Female
Connections:
- net GND: now also J4.10 (Pin_10), J4.5 (Pin_5), J4.6 (Pin_6), J4.7 (Pin_7), J4.8 (Pin_8), J4.9 (Pin_9), J5.10 (Pin_10), J5.5 (Pin_5), J5.6 (Pin_6), J5.7 (Pin_7), J5.8 (Pin_8), J5.9 (Pin_9), J8.11 (Pin_11), J8.12 (Pin_12), D?.1 (K), D?.1 (K), D?.1 (K), J?.2 (Pin_2), J?.4 (Pin_4)
- net VCC: now also MEGA2560PRO1.5V@1, MEGA2560PRO1.5V@2, 280R.1, J?.1 (Pin_1); no longer MEGA2560PRO1.VIN@1, MEGA2560PRO1.VIN@2
- net VDD: now also 1.6k.1
- net +12V: now reaches J4.11 (Pin_11)
- net +12V: now also J4.12 (Pin_12), J5.11 (Pin_11), J5.12 (Pin_12), 1k.1, J?.1 (Pin_1)
- new net: 280R.2, D?.2 (A)
- new net: 1k.2, D?.2 (A)
- new net: 1.6k.2, D?.2 (A)
- new net +3V3: J?.3 (Pin_3)
- new net +5V: J?.2 (Pin_2)
